Commit message: added comments

File: robotiq_3f_gripper_visualization/cfg/robotiq-3f-gripper_articulated_macro.xacro (robot description, xacro)
@@ -20,12 +20,12 @@
             <joint name="fixed" type="fixed">
                 <parent link="world"/>
-                <child link="base_link_hithand"/>
+                <child link="${prefix}palm"/>
                 <origin xyz="0 0 0.1" rpy="0 0 0"/>
             </joint>
         </xacro:if> -->
         <!-- <xacro:if value="${attached}">
-            <joint name="${ns}_hithand_joint" type="fixed">
+            <joint name="${ns}_robotiq_3f_joint" type="fixed">
                 <parent link="${parent}"/>
-                <child link="base_link_hithand"/>
+                <child link="${prefix}palm"/>
                 <origin xyz="${xyz}" rpy="${rpy}"/>
             </joint>
