Commit message: updated xacros

File: robotiq_3f_gripper_visualization/cfg/robotiq-3f-gripper_articulated.xacro (robot description, xacro)
@@ -7,4 +7,9 @@
         <xacro:include filename="$(find robotiq_3f_gripper_visualization)/cfg/robotiq-3f-gripper_articulated_macro.xacro" />
         <xacro:robotiq-3f-gripper_articulated prefix=""/>
+<!-- <robot xmlns:xacro="http://ros.org/wiki/xacro" name="robotiq-3f-gripper_articulated">
+        <xacro:arg name="attached"    default="false"/>
+        <xacro:arg name="parent"      default=""     />
+        <xacro:include filename="$(find robotiq_3f_gripper_visualization)/cfg/robotiq-3f-gripper_articulated_macro.xacro" />
+        <xacro:robotiq-3f-gripper_articulated prefix="" attached="$(arg attached)" parent="$(arg parent)" xyz="0 0 0" rpy="0 0 0 "/> -->
 <!--
         <xacro:include filename="$(find robotiq_3f_gripper_visualization)/cfg/robotiq-3f-gripper_finger_articulated_macro.xacro" />

File: robotiq_3f_gripper_visualization/cfg/robotiq-3f-gripper_articulated_macro.xacro (robot description, xacro)
@@ -1,2 +1,3 @@
+<?xml version="1.0" ?>
 <!--
 robotiq-3f-gripper_articulated_macro(prefix)
@@ -8,7 +9,26 @@
         <xacro:include filename="$(find robotiq_3f_gripper_visualization)/cfg/robotiq-3f-gripper_finger_articulated_macro.xacro" />
         <xacro:macro name="robotiq-3f-gripper_articulated" params="prefix">
+		<!-- <xacro:macro name="robotiq-3f-gripper_articulated" params="prefix attached:='false' parent:='' ns:='' rpy:='0 0 0' xyz:='0 0 0'"> -->
         <xacro:robotiq-3f-gripper_finger_articulated prefix="${prefix}finger_1_"/>
         <xacro:robotiq-3f-gripper_finger_articulated prefix="${prefix}finger_2_"/>
         <xacro:robotiq-3f-gripper_finger_articulated prefix="${prefix}finger_middle_"/>
+        <!-- <xacro:property name="mu1" value="0.6"/>
+        <xacro:property name="mu2" value="0.6"/> -->
+        <!-- Either attach the Hithand to the then here defined world link or attach to given robot link which itself defines the world frame -->
+        <!-- <xacro:if value="${not attached}">
+        <link name="world"/>
+            <joint name="fixed" type="fixed">
+                <parent link="world"/>
+                <child link="base_link_hithand"/>
+                <origin xyz="0 0 0.1" rpy="0 0 0"/>
+            </joint>
+        </xacro:if> -->
+        <!-- <xacro:if value="${attached}">
+            <joint name="${ns}_hithand_joint" type="fixed">
+                <parent link="${parent}"/>
+                <child link="base_link_hithand"/>
+                <origin xyz="${xyz}" rpy="${rpy}"/>
+            </joint>
+        </xacro:if> -->
 		<!-- link list -->
 		<link name="${prefix}palm">

File: robotiq_3f_gripper_visualization/cfg/robotiq-3f-gripper_finger_articulated_macro.xacro (robot description, xacro)
@@ -1,2 +1,3 @@
+<?xml version="1.0" ?>
 <!--
 robotiq-3f-gripper_finder_articulated_macro(prefix)

Commit message: added loading of articulated and normal grippers in gazebo, improved launchs and configs

File: robotiq_3f_gripper_visualization/cfg/robotiq-3f-gripper_articulated.xacro (robot description, xacro)
@@ -4,15 +4,8 @@
 3 fingered gripper.
 -->
-<robot name="robotiq-3f-gripper_articulated" xmlns:xacro="http://ros.org/wiki/xacro">
-        <xacro:include filename="$(find robotiq_3f_gripper_visualization)/cfg/robotiq-3f-gripper_articulated_macro.xacro" />
-        <xacro:robotiq-3f-gripper_articulated prefix=""/>
-<!-- <robot xmlns:xacro="http://ros.org/wiki/xacro" name="robotiq-3f-gripper_articulated">
+<robot xmlns:xacro="http://ros.org/wiki/xacro" name="robotiq-3f-gripper_articulated">
         <xacro:arg name="attached"    default="false"/>
         <xacro:arg name="parent"      default=""     />
         <xacro:include filename="$(find robotiq_3f_gripper_visualization)/cfg/robotiq-3f-gripper_articulated_macro.xacro" />
-        <xacro:robotiq-3f-gripper_articulated prefix="" attached="$(arg attached)" parent="$(arg parent)" xyz="0 0 0" rpy="0 0 0 "/> -->
-<!--
-        <xacro:include filename="$(find robotiq_3f_gripper_visualization)/cfg/robotiq-3f-gripper_finger_articulated_macro.xacro" />
-        <xacro:robotiq-3f-gripper_finger_articulated prefix=""/>
--->
+        <xacro:robotiq-3f-gripper_articulated prefix="" attached="$(arg attached)" ns="" parent="$(arg parent)" xyz="0 0 0" rpy="0 0 0"/>
 </robot>

File: robotiq_3f_gripper_visualization/cfg/robotiq-3f-gripper_articulated_macro.xacro (robot description, xacro)
@@ -6,8 +6,7 @@
 there are multiple hands then a prefix followed by an "_" is needed.
 -->
-<robot xmlns:xacro="http://ros.org/wiki/xacro">
-        <xacro:include filename="$(find robotiq_3f_gripper_visualization)/cfg/robotiq-3f-gripper_finger_articulated_macro.xacro" />
-        <xacro:macro name="robotiq-3f-gripper_articulated" params="prefix">
-		<!-- <xacro:macro name="robotiq-3f-gripper_articulated" params="prefix attached:='false' parent:='' ns:='' rpy:='0 0 0' xyz:='0 0 0'"> -->
+<robot xmlns:xacro="http://ros.org/wiki/xacro" name="robotiq-3f-gripper_articulated">
+	<xacro:include filename="$(find robotiq_3f_gripper_visualization)/cfg/robotiq-3f-gripper_finger_articulated_macro.xacro" />
+	<xacro:macro name="robotiq-3f-gripper_articulated" params="prefix attached:='true' parent:='' ns:='' rpy:='0 0 0' xyz:='0 0 0'">
         <xacro:robotiq-3f-gripper_finger_articulated prefix="${prefix}finger_1_"/>
         <xacro:robotiq-3f-gripper_finger_articulated prefix="${prefix}finger_2_"/>
@@ -24,11 +23,12 @@
             </joint>
         </xacro:if> -->
-        <!-- <xacro:if value="${attached}">
-            <joint name="${ns}_robotiq_3f_joint" type="fixed">
-                <parent link="${parent}"/>
-                <child link="${prefix}palm"/>
-                <origin xyz="${xyz}" rpy="${rpy}"/>
-            </joint>
-        </xacro:if> -->
+        <xacro:if value="${attached}">
+            <joint name="${prefix}robotiq_hand_joint" type="fixed">
+				<!-- <xacro:insert_block name="origin"/> -->
+				<parent link="${parent}"/>
+				<child link="${prefix}palm"/>
+				<origin xyz="${xyz}" rpy="${rpy}"/>
+			</joint>
+        </xacro:if>
 		<!-- link list -->
 		<link name="${prefix}palm">

File: robotiq_3f_gripper_visualization/cfg/robotiq_hand_macro.urdf.xacro (robot description, xacro)
@@ -632,11 +632,18 @@
     </gazebo>
   </xacro:macro>
-  <xacro:macro name="robotiq_hand" params="prefix *origin reflect parent">
+  <xacro:macro name="robotiq_hand" params="prefix attached reflect parent rpy:='0 0 0' xyz:='0 0 0'">
     <!-- joint attaching parent link to robotiq hand -->
-    <joint name="${prefix}robotiq_hand_joint" type="fixed">
-      <xacro:insert_block name="origin"/>
+    <!-- <joint name="${prefix}robotiq_hand_joint" type="fixed">
+      <origin xyz="${xyz}" rpy="${rpy}"/>
       <parent link="${parent}"/>
       <child link="${prefix}palm"/>
-    </joint>
+    </joint> -->
+    <xacro:if value="${attached}">
+      <joint name="${prefix}robotiq_hand_joint" type="fixed">
+        <origin xyz="${xyz}" rpy="${rpy}"/>
+        <parent link="${parent}"/>
+        <child link="${prefix}palm"/>
+      </joint>
+    </xacro:if>
     <!-- Insert the fingers -->
     <xacro:robotiq_finger prefix="${prefix}finger_1_"/>

Commit message: added proper loading of robotiq grippers

File: robotiq_3f_gripper_visualization/cfg/robotiq-3f-gripper_articulated.xacro (robot description, xacro)
@@ -6,6 +6,6 @@
 <robot xmlns:xacro="http://ros.org/wiki/xacro" name="robotiq-3f-gripper_articulated">
         <xacro:arg name="attached"    default="false"/>
-        <xacro:arg name="parent"      default=""     />
+        <xacro:arg name="parent"      default="panda_link8"     />
         <xacro:include filename="$(find robotiq_3f_gripper_visualization)/cfg/robotiq-3f-gripper_articulated_macro.xacro" />
-        <xacro:robotiq-3f-gripper_articulated prefix="" attached="$(arg attached)" ns="" parent="$(arg parent)" xyz="0 0 0" rpy="0 0 0"/>
+        <xacro:robotiq-3f-gripper_articulated prefix="left_hand" attached="$(arg attached)" ns="" parent="$(arg parent)" xyz="0 0 0" rpy="0 0 0"/>
 </robot>

File: robotiq_3f_gripper_visualization/cfg/robotiq-3f-gripper_articulated_macro.xacro (robot description, xacro)
@@ -8,5 +8,5 @@
 <robot xmlns:xacro="http://ros.org/wiki/xacro" name="robotiq-3f-gripper_articulated">
 	<xacro:include filename="$(find robotiq_3f_gripper_visualization)/cfg/robotiq-3f-gripper_finger_articulated_macro.xacro" />
-	<xacro:macro name="robotiq-3f-gripper_articulated" params="prefix attached:='true' parent:='' ns:='' rpy:='0 0 0' xyz:='0 0 0'">
+	<xacro:macro name="robotiq-3f-gripper_articulated" params="prefix attached:='true' parent ns:='' rpy:='0 0 0' xyz:='0 0 0'">
         <xacro:robotiq-3f-gripper_finger_articulated prefix="${prefix}finger_1_"/>
         <xacro:robotiq-3f-gripper_finger_articulated prefix="${prefix}finger_2_"/>
@@ -23,12 +23,12 @@
             </joint>
         </xacro:if> -->
-        <xacro:if value="${attached}">
-            <joint name="${prefix}robotiq_hand_joint" type="fixed">
-				<!-- <xacro:insert_block name="origin"/> -->
-				<parent link="${parent}"/>
-				<child link="${prefix}palm"/>
-				<origin xyz="${xyz}" rpy="${rpy}"/>
-			</joint>
-        </xacro:if>
+        <!-- <xacro:if value="${attached}"> -->
+		<joint name="${prefix}robotiq_hand_joint" type="fixed">
+			<!-- <xacro:insert_block name="origin"/> -->
+			<parent link="${parent}"/>
+			<child link="${prefix}palm"/>
+			<origin xyz="${xyz}" rpy="${rpy}"/>
+		</joint>
+        <!-- </xacro:if> -->
 		<!-- link list -->
 		<link name="${prefix}palm">

File: robotiq_3f_gripper_visualization/cfg/robotiq_hand.xacro (robot description, xacro)
@@ -6,4 +6,4 @@
 <robot name="robotiq_hand" xmlns:xacro="http://ros.org/wiki/xacro">
         <xacro:include filename="$(find robotiq_3f_gripper_visualization)/cfg/robotiq_hand_macro.urdf.xacro" />
-        <xacro:robotiq_hand prefix="" attached="false" reflect="" parent="" xyz="0 0 0" rpy="0 0 0"/>
+        <xacro:robotiq_hand prefix="left_hand" attached="false" reflect="" parent="panda_link8" xyz="0 0 0" rpy="0 0 0"/>
 </robot>

File: robotiq_3f_gripper_visualization/cfg/robotiq_hand_macro.urdf.xacro (robot description, xacro)
@@ -634,10 +634,18 @@
   <xacro:macro name="robotiq_hand" params="prefix attached reflect parent rpy:='0 0 0' xyz:='0 0 0'">
     <!-- joint attaching parent link to robotiq hand -->
-    <!-- <joint name="${prefix}robotiq_hand_joint" type="fixed">
+    <joint name="${prefix}robotiq_hand_joint" type="fixed">
       <origin xyz="${xyz}" rpy="${rpy}"/>
       <parent link="${parent}"/>
       <child link="${prefix}palm"/>
-    </joint> -->
-    <xacro:if value="${attached}">
+    </joint>
+    <!-- <xacro:if value="${not attached}">
+        <link name="world_1"/>
+            <joint name="fixed" type="fixed">
+                <parent link="world_1"/>
+                <child link="${prefix}palm"/>
+                <origin xyz="0 0 0.1" rpy="0 0 0"/>
+            </joint>
+        </xacro:if> -->
+    <!-- <xacro:if value="${attached}">
       <joint name="${prefix}robotiq_hand_joint" type="fixed">
         <origin xyz="${xyz}" rpy="${rpy}"/>
@@ -645,5 +653,5 @@
         <child link="${prefix}palm"/>
       </joint>
-    </xacro:if>
+    </xacro:if> -->
     <!-- Insert the fingers -->
     <xacro:robotiq_finger prefix="${prefix}finger_1_"/>

Commit message: mounted robotiq3f to panda robot

File: robotiq_3f_gripper_visualization/cfg/robotiq-3f-gripper_articulated.xacro (robot description, xacro)
@@ -5,7 +5,7 @@
 -->
 <robot xmlns:xacro="http://ros.org/wiki/xacro" name="robotiq-3f-gripper_articulated">
-        <xacro:arg name="attached"    default="false"/>
+        <xacro:arg name="attached"    default="true"/>
         <xacro:arg name="parent"      default="panda_link8"     />
         <xacro:include filename="$(find robotiq_3f_gripper_visualization)/cfg/robotiq-3f-gripper_articulated_macro.xacro" />
-        <xacro:robotiq-3f-gripper_articulated prefix="left_hand" attached="$(arg attached)" ns="" parent="$(arg parent)" xyz="0 0 0" rpy="0 0 0"/>
+        <xacro:robotiq-3f-gripper_articulated prefix="left_hand" attached="$(arg attached)" ns="" parent="$(arg parent)" xyz="0 0 0.05" rpy="1.5708 0 0"/>
 </robot>

File: robotiq_3f_gripper_visualization/cfg/robotiq-3f-gripper_articulated_macro.xacro (robot description, xacro)
@@ -8,5 +8,5 @@
 <robot xmlns:xacro="http://ros.org/wiki/xacro" name="robotiq-3f-gripper_articulated">
 	<xacro:include filename="$(find robotiq_3f_gripper_visualization)/cfg/robotiq-3f-gripper_finger_articulated_macro.xacro" />
-	<xacro:macro name="robotiq-3f-gripper_articulated" params="prefix attached:='true' parent ns:='' rpy:='0 0 0' xyz:='0 0 0'">
+	<xacro:macro name="robotiq-3f-gripper_articulated" params="prefix attached:='true' parent ns:='' rpy xyz">
         <xacro:robotiq-3f-gripper_finger_articulated prefix="${prefix}finger_1_"/>
         <xacro:robotiq-3f-gripper_finger_articulated prefix="${prefix}finger_2_"/>
@@ -15,5 +15,5 @@
         <xacro:property name="mu2" value="0.6"/> -->
         <!-- Either attach the Hithand to the then here defined world link or attach to given robot link which itself defines the world frame -->
-        <!-- <xacro:if value="${not attached}">
+        <xacro:if value="${not attached}">
         <link name="world"/>
             <joint name="fixed" type="fixed">
@@ -22,13 +22,13 @@
                 <origin xyz="0 0 0.1" rpy="0 0 0"/>
             </joint>
-        </xacro:if> -->
-        <!-- <xacro:if value="${attached}"> -->
-		<joint name="${prefix}robotiq_hand_joint" type="fixed">
-			<!-- <xacro:insert_block name="origin"/> -->
-			<parent link="${parent}"/>
-			<child link="${prefix}palm"/>
-			<origin xyz="${xyz}" rpy="${rpy}"/>
-		</joint>
-        <!-- </xacro:if> -->
+        </xacro:if>
+        <xacro:if value="${attached}">
+			<joint name="${prefix}robotiq_hand_joint" type="fixed">
+				<!-- <xacro:insert_block name="origin"/> -->
+				<parent link="${parent}"/>
+				<child link="${prefix}palm"/>
+				<origin xyz="${xyz}" rpy="${rpy}"/>
+			</joint>
+        </xacro:if>
 		<!-- link list -->
 		<link name="${prefix}palm">

File: robotiq_3f_gripper_visualization/cfg/robotiq_hand.xacro (robot description, xacro)
@@ -6,4 +6,4 @@
 <robot name="robotiq_hand" xmlns:xacro="http://ros.org/wiki/xacro">
         <xacro:include filename="$(find robotiq_3f_gripper_visualization)/cfg/robotiq_hand_macro.urdf.xacro" />
-        <xacro:robotiq_hand prefix="left_hand" attached="false" reflect="" parent="panda_link8" xyz="0 0 0" rpy="0 0 0"/>
+        <xacro:robotiq_hand prefix="left_hand" attached="true" reflect="" parent="panda_link8" xyz="0 0 0.05" rpy="1.5708 0 0"/>
 </robot>

File: robotiq_3f_gripper_visualization/cfg/robotiq_hand_macro.urdf.xacro (robot description, xacro)
@@ -632,20 +632,14 @@
     </gazebo>
   </xacro:macro>
-  <xacro:macro name="robotiq_hand" params="prefix attached reflect parent rpy:='0 0 0' xyz:='0 0 0'">
-    <!-- joint attaching parent link to robotiq hand -->
-    <joint name="${prefix}robotiq_hand_joint" type="fixed">
-      <origin xyz="${xyz}" rpy="${rpy}"/>
-      <parent link="${parent}"/>
-      <child link="${prefix}palm"/>
-    </joint>
-    <!-- <xacro:if value="${not attached}">
-        <link name="world_1"/>
+  <xacro:macro name="robotiq_hand" params="prefix attached reflect parent rpy xyz">
+    <xacro:if value="${not attached}">
+        <link name="world"/>
             <joint name="fixed" type="fixed">
-                <parent link="world_1"/>
+                <parent link="world"/>
                 <child link="${prefix}palm"/>
                 <origin xyz="0 0 0.1" rpy="0 0 0"/>
             </joint>
-        </xacro:if> -->
-    <!-- <xacro:if value="${attached}">
+        </xacro:if>
+    <xacro:if value="${attached}">
       <joint name="${prefix}robotiq_hand_joint" type="fixed">
         <origin xyz="${xyz}" rpy="${rpy}"/>
@@ -653,5 +647,5 @@
         <child link="${prefix}palm"/>
       </joint>
-    </xacro:if> -->
+    </xacro:if>
     <!-- Insert the fingers -->
     <xacro:robotiq_finger prefix="${prefix}finger_1_"/>
