Commit message: fixed palm transformation bug

File: robotiq_3f_gripper_visualization/cfg/robotiq_hand_macro.urdf.xacro (robot description, xacro)
@@ -683,4 +683,10 @@
         <mu2>1.1</mu2>
       </gazebo>
+    <joint name="robotiq_palm_joint" type="fixed">
+      <parent link="${prefix}palm"/>
+      <child link="palm_link_robotiq"/>
+      <origin xyz="0.02 0 0" rpy="-1.5708 0 1.5708"/>
+    </joint>
+    <link name="palm_link_robotiq"/>
     <!-- End of link list -->
     <!-- Joint list -->
